File: mp3_fa2026.kicad_pcb (KiCad board)
At the start: 2 copper layers, 21.8 x 52.6 mm, 43 parts, among them J1 USB4105-GF-A, J2 LEFT, J3 RIGHT, J4 DEBUG, U1 RP2354A, U2 MCP1702T-3302E_CB, X1 IQXO-791_12MHz

Commit message: fix C9 bypass capacitor placement
Parts:
- G***: moved to B.Cu
- moved C9 12.0 mm to (90.0, 93.5), turned to 0 degrees
- moved C3 0.18 mm to (87.6, 93.9)
- moved R6 0.08 mm to (89.3, 90.8)
- moved C12 0.05 mm to (86.8, 98.1)
- turned G*** to 180 degrees
Routing:
- net +3V3: track 96.8 -> 79.1 mm
- net GND: track 48.5 -> 47.5 mm
- net /GPIO10: track 10.3 -> 9.68 mm
